File: KiCad/dk-spot-welder.kicad_sch (KiCad schematic)
At the start: 48 parts, among them Q1 IRF1404, Q2 IRF1404, Q3 IRF1404, Q4 IRF1404, Q5 IRF1404, Q6 IRF1404, Q7 IRF1404, Q8 IRF1404, U1 MCP1407, U2 L7805, U3 ATtiny13-20P, U4 PC817

Commit message: update connections from M3 to 4mm
Parts:
- TP1, TP2, TP3: footprint TestPoint:TestPoint_Plated_Hole_D3.0mm -> MountingHole:MountingHole_4mm_Pad_Via
Changed lines of the file:
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@@
 			)
 		)
-		(property "Footprint" "TestPoint:TestPoint_Plated_Hole_D3.0mm"
+		(property "Footprint" "MountingHole:MountingHole_4mm_Pad_Via"
 			(at 36.83 69.85 0)
 			(hide yes)
@@
 			)
 		)
-		(property "Footprint" "TestPoint:TestPoint_Plated_Hole_D3.0mm"
+		(property "Footprint" "MountingHole:MountingHole_4mm_Pad_Via"
 			(at 27.94 57.15 0)
 			(hide yes)
@@
 			)
 		)
-		(property "Footprint" "TestPoint:TestPoint_Plated_Hole_D3.0mm"
+		(property "Footprint" "MountingHole:MountingHole_4mm_Pad_Via"
 			(at 162.56 25.4 0)
 			(hide yes)

Commit message: add another tp on PB5 to use with manual weld button
Parts:
- added TP5: WELD_BTN, TestPoint:TestPoint_2Pads_Pitch5.08mm_Drill1.3mm, symbol Connector:TestPoint_2Pole
- TP4: value TestPoint_2Pole -> WELD_DURATION
Connections:
- net CTRL_GND: now also TP5.2
- net PB5: now also TP5.1
Changed lines of the file:
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@@
 	)
 	(junction
+		(at 111.76 168.91)
+		(diameter 0)
+		(color 0 0 0 0)
+	)
+	(junction
 		(at 134.62 39.37)
 		(diameter 0)
@@
 		(color 0 0 0 0)
 	)
+	(junction
+		(at 147.32 173.99)
+		(diameter 0)
+		(color 0 0 0 0)
+	)
 	(wire
 		(pts
@@
 	(wire
 		(pts
+			(xy 111.76 168.91) (xy 129.54 168.91)
+		)
+		(stroke
+			(width 0)
+			(type default)
+		)
+	)
+	(wire
+		(pts
 			(xy 100.33 82.55) (xy 100.33 83.82)
 		)
@@
 	(wire
 		(pts
+			(xy 147.32 168.91) (xy 147.32 173.99)
+		)
+		(stroke
+			(width 0)
+			(type default)
+		)
+	)
+	(wire
+		(pts
 			(xy 162.56 129.54) (xy 171.45 129.54)
 		)
@@
 	(wire
 		(pts
+			(xy 139.7 168.91) (xy 147.32 168.91)
+		)
+		(stroke
+			(width 0)
+			(type default)
+		)
+	)
+	(wire
+		(pts
 			(xy 262.89 96.52) (xy 252.73 96.52)
 		)
@@
 		(in_pos_files yes)
 		(dnp no)
-		(fields_autoplaced yes)
 		(property "Reference" "TP4"
-			(at 134.62 168.91 0)
+			(at 125.476 171.196 0)
 			(show_name no)
 			(do_not_autoplace no)
@@
 			)
 		)
-		(property "Value" "TestPoint_2Pole"
-			(at 134.62 171.45 0)
+		(property "Value" "WELD_DURATION"
+			(at 136.652 171.196 0)
 			(show_name no)
 			(do_not_autoplace no)
@@
 					(unit 1)
 				)
+			)
+		)
+	)
+	(symbol
+		(lib_id "Connector:TestPoint_2Pole")
+		(at 134.62 168.91 0)
+		(unit 1)
+		(body_style 1)
+		(exclude_from_sim no)
+		(in_bom yes)
+		(on_board yes)
+		(in_pos_files yes)
+		(dnp no)
+		(property "Reference" "TP5"
+			(at 125.476 166.116 0)
+			(show_name no)
+			(do_not_autoplace no)
+			(effects
+				(font
+					(size 1.27 1.27)
+				)
+			)
+		)
+		(property "Value" "WELD_BTN"
+			(at 135.128 166.116 0)
+			(show_name no)
+			(do_not_autoplace no)
+			(effects
+				(font
+					(size 1.27 1.27)
+				)
+			)
+		)
+		(property "Footprint" "TestPoint:TestPoint_2Pads_Pitch5.08mm_Drill1.3mm"
+			(at 134.62 168.91 0)
+			(hide yes)
+			(show_name no)
+			(do_not_autoplace no)
+			(effects
+				(font
+					(size 1.27 1.27)
+				)
+			)
+		)
+		(property "Datasheet" ""
+			(at 134.62 168.91 0)
+			(hide yes)
+			(show_name no)
+			(do_not_autoplace no)
+			(effects
+				(font
+					(size 1.27 1.27)
+				)
+			)
+		)
+		(property "Description" "2-polar test point"
+			(at 134.62 168.91 0)
+			(hide yes)
+			(show_name no)
+			(do_not_autoplace no)
+			(effects
+				(font
+					(size 1.27 1.27)
+				)
+			)
+		)
+		(pin "1"
+		)
+		(pin "2"
+		)
+		(instances
+			(project "dk-spot-welder"
+				(path "/5fad44e9-5a8e-43be-858d-05b41920aa0c"
+					(reference "TP5")
+					(unit 1)
+				)
