File: KiCad/dk-spot-welder.kicad_pcb (KiCad board)
At the start: 4 copper layers, 112 x 72 mm, 51 parts, among them Q1 IRF1404, Q2 IRF1404, Q3 IRF1404, Q4 IRF1404, Q5 IRF1404, Q6 IRF1404, Q7 IRF1404, Q8 IRF1404, U1 MCP1407, U2 L7805, U3 ATtiny13-20P, U4 PC817

Commit message: redesigned vias and exposed copper
Parts:
- moved D6 0.97 mm to (181.7, 83.6)
- moved D1 0.93 mm to (112.2, 83.6)
- moved D2 0.93 mm to (135.5, 83.6)
- moved G*** 0.80 mm to (107.5, 129.8)
- moved TP5 0.78 mm to (110.0, 125.6)
- moved D3 0.74 mm to (158.5, 83.6)
- moved NT1 0.65 mm to (159.3, 96.3)
Routing:
- net GND: track 15.5 -> 15.1 mm, vias 158 -> 125
- net /OUT-: vias 405 -> 307
Other:
- board text added: "2026/07"
- board text added: "Spot Welder Rev. B"
- board text removed: "2026/06"
- board text removed: "Spot Welder Rev. A"
